File: vca/thomas-henry-vca/vca1/vca1.kicad_pcb (KiCad board)
At the start: 2 copper layers, 99.1 x 69.9 mm, 47 parts, among them J1 AudioJack2, J2 AudioJack2, J3 AudioJack2, J4 AudioJack2, J5 AudioJack2, J6 MAX OUT, J7 LINE OUT, J8 Conn_01x03, Q1 2N3906, SW1 SW_DIP_x01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

Commit message: testing
Parts:
- R17-OFFSET-TRIM1: footprint Potentiometer_THT:Potentiometer_ACP_CA9-V10_Vertical -> Potentiometer_THT:Potentiometer_Piher_PT-6-V_Vertical
- moved R17-OFFSET-TRIM1 2.88 mm to (86.5, 11.5)
Connections:
- U1 pad 4: Net-(U1-Pad4) -> -15V
Routing:
- net +15V: track 184.1 -> 187.0 mm
- net -15V: track 186.0 -> 184.2 mm
- net Net-(R15-Pad2): track 11.2 -> 10.1 mm
