File: vca/thomas-henry-vca/vca1/vca1.sch (KiCad schematic (older format))
At the start: 47 parts, among them J1 AudioJack2, J2 AudioJack2, J3 AudioJack2, J4 AudioJack2, J5 AudioJack2, J6 MAX OUT, J7 LINE OUT, J8 Conn_01x03, Q1 2N3906, SW1 SW_DIP_x01, SW2 SW_DIP_x01, SW3 SW_DIP_x01, U1 CA3080, U2 TL072, U3 TL071

Commit message: testing
Parts:
- R2: renamed from R10; value R -> 22r
- renumbered R2 to R10, R17-OFFSET-TRIM1 to R17_OFFSET_TRIM1, R18-PAD1 to R18_PAD1, R19-PAD2 to R19_PAD2, R20-PAD3 to R20_PAD3, R21-ATTEN1 to R21_ATTEN1, R22-INITIAL1 to R22_INITIAL1, R4-LEVEL1 to R4_LEVEL1
Connections:
- net -15V: now also U1.4 (V-)
- no-connect marks 0 -> 2
Changed lines of the file:
@@
 $EndComp
 $Comp
-L Device:R_POT R18-PAD1
+L Device:R_POT R18_PAD1
 U 1 1 5C7AFB57
 P 2100 1900
-F 0 "R18-PAD1" H 2030 1946 50  0000 R CNN
+F 0 "R18_PAD1" H 2030 1946 50  0000 R CNN
 F 1 "100K" H 2030 1855 50  0000 R CNN
 F 2 "Connector_PinHeader_2.54mm:PinHeader_1x03_P2.54mm_Vertical" H 2100 1900 50  0001 C CNN
@@
 $EndComp
 $Comp
-L Device:R_POT R19-PAD2
+L Device:R_POT R19_PAD2
 U 1 1 5C7B09F0
 P 2100 3250
-F 0 "R19-PAD2" H 2030 3296 50  0000 R CNN
+F 0 "R19_PAD2" H 2030 3296 50  0000 R CNN
 F 1 "100K" H 2030 3205 50  0000 R CNN
 F 2 "Connector_PinHeader_2.54mm:PinHeader_1x03_P2.54mm_Vertical" H 2100 3250 50  0001 C CNN
@@
 $EndComp
 $Comp
-L Device:R R2
+L Device:R R10
 U 1 1 5C7B09FD
 P 2600 3250
-F 0 "R2" V 2393 3250 50  0000 C CNN
+F 0 "R10" V 2393 3250 50  0000 C CNN
 F 1 "100k" V 2484 3250 50  0000 C CNN
 F 2 "Resistor_THT:R_Axial_DIN0207_L6.3mm_D2.5mm_P7.62mm_Horizontal" V 2530 3250 50  0001 C CNN
@@
 $EndComp
 $Comp
-L Device:R_POT R20-PAD3
+L Device:R_POT R20_PAD3
 U 1 1 5C7B1224
 P 2100 4600
-F 0 "R20-PAD3" H 2030 4646 50  0000 R CNN
+F 0 "R20_PAD3" H 2030 4646 50  0000 R CNN
 F 1 "100K" H 2030 4555 50  0000 R CNN
 F 2 "Connector_PinHeader_2.54mm:PinHeader_1x03_P2.54mm_Vertical" H 2100 4600 50  0001 C CNN
@@
 	4800 2000 4800 2100
 $Comp
-L Device:R_POT R17-OFFSET-TRIM1
+L Device:R_POT R17_OFFSET_TRIM1
 U 1 1 5C7B6875
 P 4300 3250
-F 0 "R17-OFFSET-TRIM1" H 4230 3296 50  0000 R CNN
+F 0 "R17_OFFSET_TRIM1" H 4230 3296 50  0000 R CNN
 F 1 "100k" H 4230 3205 50  0000 R CNN
 F 2 "Potentiometer_THT:Potentiometer_Piher_PT-6-V_Vertical" H 4300 3250 50  0001 C CNN
@@
 $EndComp
 $Comp
-L Device:R R10
+L Device:R R2
 U 1 1 5C7B6A84
 P 5150 3500
-F 0 "R10" H 5220 3546 50  0000 L CNN
-F 1 "R" H 5220 3455 50  0000 L CNN
+F 0 "R2" H 5220 3546 50  0000 L CNN
+F 1 "22r" H 5220 3455 50  0000 L CNN
 F 2 "Resistor_THT:R_Axial_DIN0207_L6.3mm_D2.5mm_P7.62mm_Horizontal" V 5080 3500 50  0001 C CNN
 F 3 "~" H 5150 3500 50  0001 C CNN
@@
 Connection ~ 4600 5000
 $Comp
-L Device:R_POT R22-INITIAL1
+L Device:R_POT R22_INITIAL1
 U 1 1 5C7D043D
 P 3850 4850
-F 0 "R22-INITIAL1" V 3643 4850 50  0000 C CNN
+F 0 "R22_INITIAL1" V 3643 4850 50  0000 C CNN
 F 1 "100K" V 3734 4850 50  0000 C CNN
 F 2 "Connector_PinHeader_2.54mm:PinHeader_1x03_P2.54mm_Vertical" H 3850 4850 50  0001 C CNN
@@
 $EndComp
 $Comp
-L Device:R_POT R21-ATTEN1
+L Device:R_POT R21_ATTEN1
 U 1 1 5C7E51BF
 P 3050 6550
-F 0 "R21-ATTEN1" H 3250 7000 50  0000 R CNN
+F 0 "R21_ATTEN1" H 3250 7000 50  0000 R CNN
 F 1 "100K" H 3150 6900 50  0000 R CNN
 F 2 "Connector_PinHeader_2.54mm:PinHeader_1x03_P2.54mm_Vertical" H 3050 6550 50  0001 C CNN
@@
 $EndComp
 $Comp
-L Device:R_POT R4-LEVEL1
+L Device:R_POT R4_LEVEL1
 U 1 1 5C84975D
 P 6950 3100
-F 0 "R4-LEVEL1" H 6880 3146 50  0000 R CNN
+F 0 "R4_LEVEL1" H 6880 3146 50  0000 R CNN
 F 1 "10K" H 6880 3055 50  0000 R CNN
 F 2 "Connector_PinHeader_2.54mm:PinHeader_1x03_P2.54mm_Vertical" H 6950 3100 50  0001 C CNN
@@
 	8000 4800 8000 4950
 Wire Wire Line
-	7750 4900 7750 5200
+	7750 4900 7750 5100
 Wire Wire Line
 	7750 4700 7850 4700
 Wire Wire Line
-	7850 4350 7850 4700
+	7850 4350 7850 4450
 $Comp
 L Amplifier_Operational:TL072 U2
@@
 Wire Wire Line
 	2000 1700 2100 1700
+$Comp
+L power:-15V #PWR0134
+U 1 1 5C9F9B96
+P 5600 1750
+F 0 "#PWR0134" H 5600 1850 50  0001 C CNN
+F 1 "-15V" H 5615 1923 50  0000 C CNN
+F 2 "" H 5600 1750 50  0001 C CNN
+F 3 "" H 5600 1750 50  0001 C CNN
+	1    5600 1750
+	1    0    0    -1
+$EndComp
+Wire Wire Line
+	5600 1750 5600 1800
+$Comp
+L power:PWR_FLAG #FLG0101
+U 1 1 5CA12885
+P 8250 4450
+F 0 "#FLG0101" H 8250 4525 50  0001 C CNN
+F 1 "PWR_FLAG" H 8250 4624 50  0000 C CNN
+F 2 "" H 8250 4450 50  0001 C CNN
+F 3 "~" H 8250 4450 50  0001 C CNN
+	1    8250 4450
+	1    0    0    -1
+$EndComp
+Wire Wire Line
+	8250 4450 7850 4450
+Connection ~ 7850 4450
+Wire Wire Line
+	7850 4450 7850 4700
+$Comp
+L power:PWR_FLAG #FLG0102
+U 1 1 5CA17C6D
+P 7500 5200
+F 0 "#FLG0102" H 7500 5275 50  0001 C CNN
+F 1 "PWR_FLAG" H 7500 5374 50  0000 C CNN
+F 2 "" H 7500 5200 50  0001 C CNN
+F 3 "~" H 7500 5200 50  0001 C CNN
+	1    7500 5200
+	1    0    0    -1
+$EndComp
+Wire Wire Line
+	7750 5100 7650 5100
+Wire Wire Line
+	7650 5100 7650 5200
+Wire Wire Line
+	7650 5200 7500 5200
+Connection ~ 7750 5100
+Wire Wire Line
+	7750 5100 7750 5200
+$Comp
+L power:PWR_FLAG #FLG0103
+U 1 1 5CA2C8FE
+P 8100 4750
+F 0 "#FLG0103" H 8100 4825 50  0001 C CNN
+F 1 "PWR_FLAG" H 8100 4924 50  0000 C CNN
+F 2 "" H 8100 4750 50  0001 C CNN
+F 3 "~" H 8100 4750 50  0001 C CNN
+	1    8100 4750
+	1    0    0    -1
+$EndComp
+Wire Wire Line
+	8100 4750 8000 4750
+Wire Wire Line
+	8000 4750 8000 4800
+Connection ~ 8000 4800
+NoConn ~ 5200 5700
+NoConn ~ 5100 5700
 $EndSCHEMATC
